Commit message: Fix gripper calibration, packet parsing, motor disable, and tune URDF masses
- Fix gripper calibration: send VEL command once then poll with refresh
  frames (matching Python), raise torque threshold to 1.2, add timeout
- Fix packet parsing: filter parameter response packets (data[2]==0x33/0x55)
  that were misinterpreted as motor state, drain serial buffer before
  reading initial positions
- Fix motor disable on shutdown: proper delays, works for all modes
- Add disable_torque_on_disconnect config option through full stack
  (C++ RtLoopConfig → DK1RobotConfig → DK1FollowerConfig → teleop CLI)
- Remove debug logging from RT loop (first-20-cycles logging)
- Tune URDF link masses based on bi-directional gravity measurement:
  link4-5: 0.3995→0.42, link5-6: 0.4121→0.433, link6-7: 0.5→0.54
- Rewrite measure_gravity.py with bi-directional friction-cancelling method

Co-Authored-By: Claude Opus 4.6 <noreply@anthropic.com>

File: urdf/follower/TRLC-DK1-Follower.urdf (robot description, URDF)
Before this commit: robot TRLC-DK1-Follower, 11 links, 10 joints
Links:
- link link4-5: mass 0.3995 -> 0.42
- link link5-6: mass 0.4121 -> 0.433
- link link6-7: mass 0.5 -> 0.54

Commit message: Rename tool0 link to tcp and add flange tool0 frame
The previous tool0 link sat at the +0.158m fingertip grasp point, which is
semantically the TCP, not the ROS-Industrial flange frame. Rename it to tcp
and add a separate tool0 at the link6-7 (flange) origin so cartesian actions
can use a zero-lever effector frame decoupled from wrist-rotation lever.

Co-Authored-By: Claude Opus 4.8 (1M context) <noreply@anthropic.com>

File: urdf/follower/TRLC-DK1-Follower.urdf (robot description, URDF)
Before this commit: robot TRLC-DK1-Follower, 11 links, 10 joints
Links:
- added link tcp
Joints:
- removed joint gripper_tool0
- added joint tcp_joint: type fixed, parent link6-7, child tcp, origin xyz=0.158 0 0 rpy=-1.5707963267948966 0 -1.5707963267948966
- added joint tool0_joint: type fixed, parent link6-7, child tool0, origin xyz=0 0 0 rpy=-1.5707963267948966 0 -1.5707963267948966

Commit message: Restructure effector frames: tool0 at flange, tcp at grasp point
The previous tool0 link sat at the +0.158m fingertip plane, which is neither
the ROS-Industrial flange frame nor the actual grasp point. Restructure into
two frames:

- tool0 = flange (ROS-Industrial convention): link6-7 origin with OpenCV
  orientation (z=approach/front, x=right). Zero-lever effector frame for
  cartesian actions, decoupling position deltas from wrist-rotation lever.
- tcp = grasp point, child of tool0 at z=0.153: 5mm before the finger tips
  (tips are at 0.158).

With tcp as a child of tool0, its offset is a pure translation along tool-z
and the orientation convention is defined in exactly one place.

Co-Authored-By: Claude Opus 4.8 (1M context) <noreply@anthropic.com>

File: urdf/follower/TRLC-DK1-Follower.urdf (robot description, URDF)
Before this commit: robot TRLC-DK1-Follower, 11 links, 10 joints
Links:
- added link tcp
Joints:
- removed joint gripper_tool0
- added joint tcp_joint: type fixed, parent tool0, child tcp, origin xyz=0 0 0.153 rpy=0 0 0
- added joint tool0_joint: type fixed, parent link6-7, child tool0, origin xyz=0 0 0 rpy=-1.5707963267948966 0 -1.5707963267948966

Commit message: Move tcp to grasp point 5mm before finger tips; add fingertips_center
Restructure effector frames: tcp and fingertips_center are now children of
tool0, so their offsets are pure translations along tool-z (approach) and the
OpenCV orientation convention is defined in exactly one place (tool0_joint).

tcp moves from the geometric finger tip plane (0.158) to the grasp point 5mm
before the tips (0.153); fingertips_center keeps the tip plane at 0.158 for
clearance checks / pre-grasp approach.

Co-Authored-By: Claude Opus 4.8 (1M context) <noreply@anthropic.com>

File: urdf/follower/TRLC-DK1-Follower.urdf (robot description, URDF)
Before this commit: robot TRLC-DK1-Follower, 12 links, 11 joints
Links:
- added link fingertips_center
Joints:
- added joint fingertips_center_joint: type fixed, parent tool0, child fingertips_center, origin xyz=0 0 0.158 rpy=0 0 0
- joint tcp_joint: origin xyz=0.158 0 0 rpy=-1.5707963267948966 0 -1.5707963267948966 -> xyz=0 0 0.153 rpy=0 0 0; parent link6-7 -> tool0

Commit message: Remove fingertips_center frame; note tip plane in tcp comment
Only 5mm from tcp — consumers compute offsets along tool-z from tcp anyway,
and two near-identical effector frames invite ambiguity about the canonical
action frame. The tip plane (0.158) is documented in the tcp comment.

Co-Authored-By: Claude Opus 4.8 (1M context) <noreply@anthropic.com>

File: urdf/follower/TRLC-DK1-Follower.urdf (robot description, URDF)
Before this commit: robot TRLC-DK1-Follower, 13 links, 12 joints
Links:
- removed link fingertips_center
Joints:
- removed joint fingertips_center_joint
